File: smd-challenge.kicad_sch (KiCad schematic)
At the start: 25 parts, among them J1 DX07S016JA1R1500, J2 Conn_01x05, U1 MIC5504-3.3YM5, U2 ATSAMD21E15B-M, Y1 FA-238 16.0000MB-K3

Commit message: Add pull-up resistor on SWCLK per Microchip docs
Parts:
- added R9: 1k, Resistor_SMD:R_0603_1608Metric, symbol Device:R
Connections:
- net +3V3: now also R9.1
- net SWCLK: now also R9.2
Changed lines of the file:
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@@
   (junction (at 59.69 29.21) (diameter 0.9144) (color 0 0 0 0))
   (junction (at 73.66 143.51) (diameter 0.9144) (color 0 0 0 0))
+  (junction (at 98.806 123.19) (diameter 0.9144) (color 0 0 0 0))
   (junction (at 130.81 27.94) (diameter 0.9144) (color 0 0 0 0))
   (junction (at 135.89 27.94) (diameter 0.9144) (color 0 0 0 0))
@@
     (stroke (width 0) (type solid) (color 0 0 0 0))
   )
+  (wire (pts (xy 90.932 123.19) (xy 98.806 123.19))
+    (stroke (width 0) (type solid) (color 0 0 0 0))
+  )
+  (wire (pts (xy 98.806 123.19) (xy 110.49 123.19))
+    (stroke (width 0) (type solid) (color 0 0 0 0))
+  )
   (wire (pts (xy 106.68 130.81) (xy 110.49 130.81))
     (stroke (width 0) (type solid) (color 0 0 0 0))
@@
     (stroke (width 0) (type solid) (color 0 0 0 0))
   )
-  (wire (pts (xy 107.95 123.19) (xy 110.49 123.19))
-    (stroke (width 0) (type solid) (color 0 0 0 0))
-  )
   (wire (pts (xy 107.95 125.73) (xy 110.49 125.73))
     (stroke (width 0) (type solid) (color 0 0 0 0))
@@
     (effects (font (size 1.27 1.27)) (justify right bottom))
   )
+  (label "SWCLK" (at 90.932 123.19 180)
+    (effects (font (size 1.27 1.27)) (justify right bottom))
+  )
   (label "NRST" (at 106.68 130.81 180)
     (effects (font (size 1.27 1.27)) (justify right bottom))
@@
   )
   (label "BLUE" (at 107.95 57.15 180)
-    (effects (font (size 1.27 1.27)) (justify right bottom))
-  )
-  (label "SWCLK" (at 107.95 123.19 180)
     (effects (font (size 1.27 1.27)) (justify right bottom))
   )
@@
     (pin "1")
   )
+  (symbol (lib_id "power:+3.3V") (at 98.806 115.57 0) (unit 1)
+    (in_bom yes) (on_board yes)
+    (property "Reference" "#PWR0102" (id 0) (at 98.806 119.38 0)
+      (effects (font (size 1.27 1.27)) hide)
+    )
+    (property "Value" "+3.3V" (id 1) (at 98.806 111.76 0))
+    (property "Footprint" "" (id 2) (at 98.806 115.57 0)
+      (effects (font (size 1.27 1.27)) hide)
+    )
+    (property "Datasheet" "" (id 3) (at 98.806 115.57 0)
+      (effects (font (size 1.27 1.27)) hide)
+    )
+    (pin "1")
+  )
   (symbol (lib_id "power:+3.3V") (at 130.81 24.13 0) (unit 1)
     (in_bom yes) (on_board yes)
@@
     )
     (property "Datasheet" "~" (id 3) (at 78.74 137.16 0)
+      (effects (font (size 1.27 1.27)) hide)
+    )
+    (pin "1")
+    (pin "2")
+  )
+  (symbol (lib_id "Device:R") (at 98.806 119.38 0) (unit 1)
+    (in_bom yes) (on_board yes)
+    (property "Reference" "R9" (id 0) (at 101.6 118.7449 0)
+      (effects (font (size 1.27 1.27)) (justify left))
+    )
+    (property "Value" "1k" (id 1) (at 101.6 121.2849 0)
+      (effects (font (size 1.27 1.27)) (justify left))
+    )
+    (property "Footprint" "Resistor_SMD:R_0603_1608Metric" (id 2) (at 97.028 119.38 90)
+      (effects (font (size 1.27 1.27)) hide)
+    )
+    (property "Datasheet" "~" (id 3) (at 98.806 119.38 0)
       (effects (font (size 1.27 1.27)) hide)
     )
@@
       (reference "#PWR0101") (unit 1) (value "+3.3V") (footprint "")
     )
+    (path "/3664deda-c085-452a-aed0-f2c419b60074"
+      (reference "#PWR0102") (unit 1) (value "+3.3V") (footprint "")
+    )
     (path "/c5fa86be-8e49-41ac-91b5-adef14ae477a"
       (reference "C1") (unit 1) (value "10u") (footprint "Capacitor_SMD:C_1206_3216Metric")
@@
       (reference "R8") (unit 1) (value "80") (footprint "Resistor_SMD:R_0201_0603Metric")
     )
+    (path "/967f5d8f-b9f3-40ec-9e84-4fa4eb7ff262"
+      (reference "R9") (unit 1) (value "1k") (footprint "Resistor_SMD:R_0603_1608Metric")
+    )
     (path "/5a44c263-eb6c-4a3d-9ffe-d3f0be38b7e7"

Commit message: Label the LEDs by color
Parts:
- D1: value LED -> RED
- D2: value LED -> ORANGE
- D3: value LED -> YELLOW
- D4: value LED -> GREEN
- D5: value LED -> BLUE
Changed lines of the file:
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@@
     (in_bom yes) (on_board yes)
     (property "Reference" "D1" (id 0) (at 194.5005 52.07 0))
-    (property "Value" "LED" (id 1) (at 194.5005 54.61 0))
+    (property "Value" "RED" (id 1) (at 194.5005 54.61 0))
     (property "Footprint" "LED_SMD:LED_1206_3216Metric" (id 2) (at 194.31 58.42 0)
       (effects (font (size 1.27 1.27)) hide)
@@
     (in_bom yes) (on_board yes)
     (property "Reference" "D2" (id 0) (at 194.5005 63.5 0))
-    (property "Value" "LED" (id 1) (at 194.5005 66.04 0))
+    (property "Value" "ORANGE" (id 1) (at 194.5005 66.04 0))
     (property "Footprint" "LED_SMD:LED_0805_2012Metric" (id 2) (at 194.31 69.85 0)
       (effects (font (size 1.27 1.27)) hide)
@@
     (in_bom yes) (on_board yes)
     (property "Reference" "D3" (id 0) (at 194.5005 73.66 0))
-    (property "Value" "LED" (id 1) (at 194.5005 76.2 0))
+    (property "Value" "YELLOW" (id 1) (at 194.5005 76.2 0))
     (property "Footprint" "LED_SMD:LED_0603_1608Metric" (id 2) (at 194.31 80.01 0)
       (effects (font (size 1.27 1.27)) hide)
@@
     (in_bom yes) (on_board yes)
     (property "Reference" "D4" (id 0) (at 194.5005 85.09 0))
-    (property "Value" "LED" (id 1) (at 194.5005 87.63 0))
+    (property "Value" "GREEN" (id 1) (at 194.5005 87.63 0))
     (property "Footprint" "LED_SMD:LED_0402_1005Metric" (id 2) (at 194.31 91.44 0)
       (effects (font (size 1.27 1.27)) hide)
@@
     (in_bom yes) (on_board yes)
     (property "Reference" "D5" (id 0) (at 194.5005 96.52 0))
-    (property "Value" "LED" (id 1) (at 194.5005 99.06 0))
+    (property "Value" "BLUE" (id 1) (at 194.5005 99.06 0))
     (property "Footprint" "LED_SMD:LED_0201_0603Metric" (id 2) (at 194.31 102.87 0)
       (effects (font (size 1.27 1.27)) hide)
@@
     )
     (path "/4334957c-4ad1-4803-b6da-6b94019f9548"
-      (reference "D1") (unit 1) (value "LED") (footprint "LED_SMD:LED_1206_3216Metric")
+      (reference "D1") (unit 1) (value "RED") (footprint "LED_SMD:LED_1206_3216Metric")
     )
     (path "/e4ea8c08-0a2c-4e29-a897-2c7cfa24998f"
-      (reference "D2") (unit 1) (value "LED") (footprint "LED_SMD:LED_0805_2012Metric")
+      (reference "D2") (unit 1) (value "ORANGE") (footprint "LED_SMD:LED_0805_2012Metric")
     )
     (path "/6d942e00-ecbe-449d-b6f5-782a89913cf0"
-      (reference "D3") (unit 1) (value "LED") (footprint "LED_SMD:LED_0603_1608Metric")
+      (reference "D3") (unit 1) (value "YELLOW") (footprint "LED_SMD:LED_0603_1608Metric")
     )
     (path "/0064dc73-b6ba-4951-a9d4-37b6018b0837"
-      (reference "D4") (unit 1) (value "LED") (footprint "LED_SMD:LED_0402_1005Metric")
+      (reference "D4") (unit 1) (value "GREEN") (footprint "LED_SMD:LED_0402_1005Metric")
     )
     (path "/3399912c-fe4d-470e-a70d-14af25b95d4f"
-      (reference "D5") (unit 1) (value "LED") (footprint "LED_SMD:LED_0201_0603Metric")
+      (reference "D5") (unit 1) (value "BLUE") (footprint "LED_SMD:LED_0201_0603Metric")
     )
     (path "/299c51ae-25e2-4f98-949f-a326091497b6"

Commit message: Swap crystal (and load caps) for what's in stock at Mouser
Parts:
- C2, C3: value 12p -> 28p
- Y1: value FA-238 16.0000MB-K3 -> ECS-160-18-33QZ-ADS-TR
Changed lines of the file:
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@@
       (effects (font (size 1.27 1.27)) (justify left))
     )
-    (property "Value" "12p" (id 1) (at 34.9251 68.58 0)
+    (property "Value" "28p" (id 1) (at 34.9251 68.58 0)
       (effects (font (size 1.27 1.27)) (justify left))
     )
@@
       (effects (font (size 1.27 1.27)) (justify left))
     )
-    (property "Value" "12p" (id 1) (at 34.9251 88.9 0)
+    (property "Value" "28p" (id 1) (at 34.9251 88.9 0)
       (effects (font (size 1.27 1.27)) (justify left))
     )
@@
       (effects (font (size 1.27 1.27)) (justify right))
     )
-    (property "Value" "FA-238 16.0000MB-K3" (id 1) (at 53.34 75.5649 90)
+    (property "Value" " ECS-160-18-33QZ-ADS-TR" (id 1) (at 53.34 75.5649 90)
       (effects (font (size 1.27 1.27)) (justify right))
     )
@@
     )
     (path "/6fd26f11-f126-405d-a547-5045b7a9c6e1"
-      (reference "C2") (unit 1) (value "12p") (footprint "Capacitor_SMD:C_0603_1608Metric")
+      (reference "C2") (unit 1) (value "28p") (footprint "Capacitor_SMD:C_0603_1608Metric")
     )
     (path "/8b358330-234f-4b1c-9989-6037fd57d4c0"
-      (reference "C3") (unit 1) (value "12p") (footprint "Capacitor_SMD:C_0603_1608Metric")
+      (reference "C3") (unit 1) (value "28p") (footprint "Capacitor_SMD:C_0603_1608Metric")
     )
     (path "/9b0d978d-5b6e-428d-b6f0-df8ac7dbe5a8"
@@
     )
     (path "/ed4d4007-899f-48cd-9839-2ec406105b44"
-      (reference "Y1") (unit 1) (value "FA-238 16.0000MB-K3") (footprint "Crystal:Crystal_SMD_SeikoEpson_FA238-4Pin_3.2x2.5mm")
-    )
-  )
+      (reference "Y1") (unit 1) (value " ECS-160-18-33QZ-ADS-TR") (footprint "Crystal:Crystal_SMD_SeikoEpson_FA238-4Pin_3.2x2.5mm")
+    )
+  )
